Commit message: 0112_1000_备份

File: src/q1_controller/urdf/Q1/urdf/Q1_wo_hand.urdf (robot description, URDF)
Before this commit: robot Q1_urdf, 31 links, 30 joints
Links:
- link L_ankle_pitch_link: geometry collision cylinder length=0.001 radius=0.001; visual mesh filename=file:///home/niic/RL_control/Q1_control/src/q1_controller/u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
- link L_ankle_roll_link: geometry collision cylinder length=0.2 radius=0.004; collision cylinder length=0.2 radius=0.004
- link L_elbow_link: geometry collision cylinder length=0.07 radius=0.04; visual mesh filename=file:///home/niic/RL_control/Q1_control/src/q1_controller/u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
- link L_forearm_yaw_link: geometry collision cylinder length=0.13 radius=0.035; visual mesh filename=file:///home/niic/RL_control/Q1_control/src/q1_controller/u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
- link L_hip_pitch_link: geometry collision cylinder length=0.18 radius=0.045; visual mesh filename=file:///home/niic/RL_control/Q1_control/src/q1_controller/u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
- link L_hip_roll_link: geometry collision cylinder length=0.07 radius=0.05; visual mesh filename=file:///home/niic/RL_control/Q1_control/src/q1_controller/u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
- link L_hip_yaw_link: geometry collision cylinder length=0.09 radius=0.045; visual mesh filename=file:///home/niic/RL_control/Q1_control/src/q1_controller/u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
- link L_knee_link: geometry collision cylinder length=0.1 radius=0.025; collision cylinder length=0.1 radius=0.065
- link L_shoulder_pitch_link: geometry collision cylinder length=0.07 radius=0.045; visual mesh filename=file:///home/niic/RL_control/Q1_control/src/q1_controller/u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
- link L_shoulder_roll_link: geometry collision cylinder length=0.07 radius=0.04; visual mesh filename=file:///home/niic/RL_control/Q1_control/src/q1_controller/u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
- link L_shoulder_yaw_link: geometry collision cylinder length=0.07 radius=0.04; visual mesh filename=file:///home/niic/RL_control/Q1_control/src/q1_controller/u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
- link L_wrist_pitch_link: geometry collision box size=0.06 0.03 0.18; visual mesh filename=file:///home/niic/RL_control/Q1_control/src/q1_controller/u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
- link L_wrist_roll_link: geometry collision cylinder length=0.01 radius=0.015; visual mesh filename=file:///home/niic/RL_control/Q1_control/src/q1_controller/u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
- link R_ankle_pitch_link: geometry collision cylinder length=0.001 radius=0.001; visual mesh filename=file:///home/niic/RL_control/Q1_control/src/q1_controller/u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
- link R_ankle_roll_link: geometry collision cylinder length=0.2 radius=0.004; collision cylinder length=0.2 radius=0.004
- link R_elbow_link: geometry collision cylinder length=0.07 radius=0.04; visual mesh filename=file:///home/niic/RL_control/Q1_control/src/q1_controller/u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
- link R_forearm_yaw_link: geometry collision cylinder length=0.13 radius=0.035; visual mesh filename=file:///home/niic/RL_control/Q1_control/src/q1_controller/u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
- link R_hip_pitch_link: geometry collision cylinder length=0.18 radius=0.045; visual mesh filename=file:///home/niic/RL_control/Q1_control/src/q1_controller/u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
- link R_hip_roll_link: geometry collision cylinder length=0.07 radius=0.05; visual mesh filename=file:///home/niic/RL_control/Q1_control/src/q1_controller/u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
- link R_hip_yaw_link: geometry collision cylinder length=0.09 radius=0.045; visual mesh filename=file:///home/niic/RL_control/Q1_control/src/q1_controller/u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
- link R_knee_link: geometry collision cylinder length=0.1 radius=0.025; collision cylinder length=0.1 radius=0.065
- link R_shoulder_pitch_link: geometry collision cylinder length=0.07 radius=0.045; visual mesh filename=file:///home/niic/RL_control/Q1_control/src/q1_controller/u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
- link R_shoulder_roll_link: geometry collision cylinder length=0.07 radius=0.04; visual mesh filename=file:///home/niic/RL_control/Q1_control/src/q1_controller/u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
- link R_shoulder_yaw_link: geometry collision cylinder length=0.07 radius=0.04; visual mesh filename=file:///home/niic/RL_control/Q1_control/src/q1_controller/u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
- link R_wrist_pitch_link: geometry collision box size=0.06 0.03 0.18; visual mesh filename=file:///home/niic/RL_control/Q1_control/src/q1_controller/u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
- link R_wrist_roll_link: geometry collision cylinder length=0.01 radius=0.015; visual mesh filename=file:///home/niic/RL_control/Q1_control/src/q1_controller/u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
- link head_pitch_link: geometry collision box size=0.01 0.12 0.12; visual mesh filename=file:///home/niic/RL_control/Q1_control/src/q1_controller/u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
- link head_yaw_link: geometry collision box size=0.01 0.01 0.01; visual mesh filename=file:///home/niic/RL_control/Q1_control/src/q1_controller/u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
- link pelvis_link: geometry collision box size=0.08 0.35 0.1; visual mesh filename=file:///home/niic/RL_control/Q1_control/src/q1_controller/u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
- link torso_link: geometry collision box size=0.16 0.16 0.4; visual mesh filename=file:///home/niic/RL_control/Q1_control/src/q1_controller/u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

Commit message: 0327_0925_git save

File: src/q1_controller/urdf/Q1/urdf/Q1_wo_hand.urdf (robot description, URDF)
Before this commit: robot Q1_urdf, 31 links, 30 joints
Links:
- link L_ankle_pitch_link: geometry collision cylinder length=0.001 radius=0.001; visual mesh filename=file:///home/hpx/HPX_Loco_3/pack/Q1_control_0203_1944/src/q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
- link L_ankle_roll_link: geometry collision cylinder length=0.2 radius=0.004; collision cylinder length=0.2 radius=0.004
- link L_elbow_link: geometry collision cylinder length=0.07 radius=0.04; visual mesh filename=file:///home/hpx/HPX_Loco_3/pack/Q1_control_0203_1944/src/q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
- link L_forearm_yaw_link: geometry collision cylinder length=0.13 radius=0.035; visual mesh filename=file:///home/hpx/HPX_Loco_3/pack/Q1_control_0203_1944/src/q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
- link L_hip_pitch_link: geometry collision cylinder length=0.18 radius=0.045; visual mesh filename=file:///home/hpx/HPX_Loco_3/pack/Q1_control_0203_1944/src/q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
- link L_hip_roll_link: geometry collision cylinder length=0.07 radius=0.05; visual mesh filename=file:///home/hpx/HPX_Loco_3/pack/Q1_control_0203_1944/src/q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
- link L_hip_yaw_link: geometry collision cylinder length=0.09 radius=0.045; visual mesh filename=file:///home/hpx/HPX_Loco_3/pack/Q1_control_0203_1944/src/q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
- link L_knee_link: geometry collision cylinder length=0.1 radius=0.025; collision cylinder length=0.1 radius=0.065
- link L_shoulder_pitch_link: geometry collision cylinder length=0.07 radius=0.045; visual mesh filename=file:///home/hpx/HPX_Loco_3/pack/Q1_control_0203_1944/src/q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
- link L_shoulder_roll_link: geometry collision cylinder length=0.07 radius=0.04; visual mesh filename=file:///home/hpx/HPX_Loco_3/pack/Q1_control_0203_1944/src/q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
- link L_shoulder_yaw_link: geometry collision cylinder length=0.07 radius=0.04; visual mesh filename=file:///home/hpx/HPX_Loco_3/pack/Q1_control_0203_1944/src/q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
- link L_wrist_pitch_link: geometry collision box size=0.06 0.03 0.18; visual mesh filename=file:///home/hpx/HPX_Loco_3/pack/Q1_control_0203_1944/src/q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
- link L_wrist_roll_link: geometry collision cylinder length=0.01 radius=0.015; visual mesh filename=file:///home/hpx/HPX_Loco_3/pack/Q1_control_0203_1944/src/q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
- link R_ankle_pitch_link: geometry collision cylinder length=0.001 radius=0.001; visual mesh filename=file:///home/hpx/HPX_Loco_3/pack/Q1_control_0203_1944/src/q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
- link R_ankle_roll_link: geometry collision cylinder length=0.2 radius=0.004; collision cylinder length=0.2 radius=0.004
- link R_elbow_link: geometry collision cylinder length=0.07 radius=0.04; visual mesh filename=file:///home/hpx/HPX_Loco_3/pack/Q1_control_0203_1944/src/q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
- link R_forearm_yaw_link: geometry collision cylinder length=0.13 radius=0.035; visual mesh filename=file:///home/hpx/HPX_Loco_3/pack/Q1_control_0203_1944/src/q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
- link R_hip_pitch_link: geometry collision cylinder length=0.18 radius=0.045; visual mesh filename=file:///home/hpx/HPX_Loco_3/pack/Q1_control_0203_1944/src/q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
- link R_hip_roll_link: geometry collision cylinder length=0.07 radius=0.05; visual mesh filename=file:///home/hpx/HPX_Loco_3/pack/Q1_control_0203_1944/src/q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
- link R_hip_yaw_link: geometry collision cylinder length=0.09 radius=0.045; visual mesh filename=file:///home/hpx/HPX_Loco_3/pack/Q1_control_0203_1944/src/q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
- link R_knee_link: geometry collision cylinder length=0.1 radius=0.025; collision cylinder length=0.1 radius=0.065
- link R_shoulder_pitch_link: geometry collision cylinder length=0.07 radius=0.045; visual mesh filename=file:///home/hpx/HPX_Loco_3/pack/Q1_control_0203_1944/src/q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
- link R_shoulder_roll_link: geometry collision cylinder length=0.07 radius=0.04; visual mesh filename=file:///home/hpx/HPX_Loco_3/pack/Q1_control_0203_1944/src/q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
- link R_shoulder_yaw_link: geometry collision cylinder length=0.07 radius=0.04; visual mesh filename=file:///home/hpx/HPX_Loco_3/pack/Q1_control_0203_1944/src/q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
- link R_wrist_pitch_link: geometry collision box size=0.06 0.03 0.18; visual mesh filename=file:///home/hpx/HPX_Loco_3/pack/Q1_control_0203_1944/src/q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
- link R_wrist_roll_link: geometry collision cylinder length=0.01 radius=0.015; visual mesh filename=file:///home/hpx/HPX_Loco_3/pack/Q1_control_0203_1944/src/q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
- link head_pitch_link: geometry collision box size=0.01 0.12 0.12; visual mesh filename=file:///home/hpx/HPX_Loco_3/pack/Q1_control_0203_1944/src/q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
- link head_yaw_link: geometry collision box size=0.01 0.01 0.01; visual mesh filename=file:///home/hpx/HPX_Loco_3/pack/Q1_control_0203_1944/src/q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
- link pelvis_link: geometry collision box size=0.08 0.35 0.1; visual mesh filename=file:///home/hpx/HPX_Loco_3/pack/Q1_control_0203_1944/src/q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
- link torso_link: geometry collision box size=0.16 0.16 0.4; visual mesh filename=file:///home/hpx/HPX_Loco_3/pack/Q1_control_0203_1944/src/q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
